File: pcb/pcb.sch (KiCad schematic (older format))
At the start: 45 parts, among them J1 LEFT, J2 LEFT-EXT, J3 RIGHT, J4 RIGHT-EXT, J5 EXT POWER, J6 RJ45, J7 RJ45, SW1 Reset, SW2 Factory Reset, SW3 User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

Commit message: :pencil: Initial pass at firmware and updates to the PCB.
Parts:
- added C13: 100nF, Capacitor_SMD:C_0603_1608Metric, symbol Device:C_Small
- D3: value CAN RX -> CAN TX
- D4: value CAN TX -> CAN RX
Connections:
- net +3V3: now also C13.2
- net CAN-RX: now also U4.5 (+); no longer U4.3 (+)
- net CAN-TX: now also U4.3 (+); no longer U4.5 (+)
- net GND: now also C13.1
Changed lines of the file:
@@
 CAN-L
 $Comp
-L power:GND #PWR051
+L power:GND #PWR052
 U 1 1 5FB00534
 P 10050 2700
-F 0 "#PWR051" H 10050 2450 50  0001 C CNN
+F 0 "#PWR052" H 10050 2450 50  0001 C CNN
 F 1 "GND" V 10055 2572 50  0000 R CNN
 F 2 "" H 10050 2700 50  0001 C CNN
@@
 $EndComp
 $Comp
-L power:GND #PWR050
+L power:GND #PWR051
 U 1 1 5FB010AC
 P 10050 2400
-F 0 "#PWR050" H 10050 2150 50  0001 C CNN
+F 0 "#PWR051" H 10050 2150 50  0001 C CNN
 F 1 "GND" V 10055 2272 50  0000 R CNN
 F 2 "" H 10050 2400 50  0001 C CNN
@@
 $EndComp
 $Comp
-L power:GND #PWR049
+L power:GND #PWR050
 U 1 1 5FB0172B
 P 10050 2300
-F 0 "#PWR049" H 10050 2050 50  0001 C CNN
+F 0 "#PWR050" H 10050 2050 50  0001 C CNN
 F 1 "GND" V 10055 2172 50  0000 R CNN
 F 2 "" H 10050 2300 50  0001 C CNN
@@
 ALT-B
 $Comp
-L power:VDDA #PWR048
+L power:VDDA #PWR049
 U 1 1 5FB02293
 P 10050 2200
-F 0 "#PWR048" H 10050 2050 50  0001 C CNN
+F 0 "#PWR049" H 10050 2050 50  0001 C CNN
 F 1 "VDDA" V 10050 2300 50  0000 L CNN
 F 2 "" H 10050 2200 50  0001 C CNN
@@
 CAN-L
 $Comp
-L power:GND #PWR047
+L power:GND #PWR048
 U 1 1 5FB02C04
 P 10050 1550
-F 0 "#PWR047" H 10050 1300 50  0001 C CNN
+F 0 "#PWR048" H 10050 1300 50  0001 C CNN
 F 1 "GND" V 10055 1422 50  0000 R CNN
 F 2 "" H 10050 1550 50  0001 C CNN
@@
 $EndComp
 $Comp
-L power:GND #PWR046
+L power:GND #PWR047
 U 1 1 5FB02C0E
 P 10050 1250
-F 0 "#PWR046" H 10050 1000 50  0001 C CNN
+F 0 "#PWR047" H 10050 1000 50  0001 C CNN
 F 1 "GND" V 10055 1122 50  0000 R CNN
 F 2 "" H 10050 1250 50  0001 C CNN
@@
 $EndComp
 $Comp
-L power:GND #PWR045
+L power:GND #PWR046
 U 1 1 5FB02C18
 P 10050 1150
-F 0 "#PWR045" H 10050 900 50  0001 C CNN
+F 0 "#PWR046" H 10050 900 50  0001 C CNN
 F 1 "GND" V 10055 1022 50  0000 R CNN
 F 2 "" H 10050 1150 50  0001 C CNN
@@
 ALT-B
 $Comp
-L power:VDDA #PWR044
+L power:VDDA #PWR045
 U 1 1 5FB02C24
 P 10050 1050
-F 0 "#PWR044" H 10050 900 50  0001 C CNN
+F 0 "#PWR045" H 10050 900 50  0001 C CNN
 F 1 "VDDA" V 10050 1150 50  0000 L CNN
 F 2 "" H 10050 1050 50  0001 C CNN
@@
 $EndComp
 $Comp
-L power:+5V #PWR040
+L power:+5V #PWR041
 U 1 1 5FB05EDC
 P 8550 1600
-F 0 "#PWR040" H 8550 1450 50  0001 C CNN
+F 0 "#PWR041" H 8550 1450 50  0001 C CNN
 F 1 "+5V" H 8565 1773 50  0000 C CNN
 F 2 "" H 8550 1600 50  0001 C CNN
@@
 $EndComp
 $Comp
-L power:GND #PWR052
+L power:GND #PWR053
 U 1 1 5FB138B1
 P 10200 4000
-F 0 "#PWR052" H 10200 3750 50  0001 C CNN
+F 0 "#PWR053" H 10200 3750 50  0001 C CNN
 F 1 "GND" H 10200 3850 50  0000 C CNN
 F 2 "" H 10200 4000 50  0001 C CNN
@@
 P 8900 4450
 F 0 "D4" H 8900 4685 50  0000 C CNN
-F 1 "CAN TX" H 8900 4594 50  0000 C CNN
+F 1 "CAN RX" H 8900 4594 50  0000 C CNN
 F 2 "LED_SMD:LED_0603_1608Metric" V 8900 4450 50  0001 C CNN
 F 3 "~" V 8900 4450 50  0001 C CNN
@@
 $EndComp
 $Comp
-L Device:LED_Small D3
-U 1 1 5FAF24A0
-P 8900 3750
-F 0 "D3" H 8900 3985 50  0000 C CNN
-F 1 "CAN RX" H 8900 3894 50  0000 C CNN
-F 2 "LED_SMD:LED_0603_1608Metric" V 8900 3750 50  0001 C CNN
-F 3 "~" V 8900 3750 50  0001 C CNN
-	1    8900 3750
-	1    0    0    -1
-$EndComp
-$Comp
-L power:+3V3 #PWR042
+L power:+3V3 #PWR043
 U 1 1 5FAF2C5F
 P 9200 3750
-F 0 "#PWR042" H 9200 3600 50  0001 C CNN
+F 0 "#PWR043" H 9200 3600 50  0001 C CNN
 F 1 "+3V3" H 9200 3900 50  0000 C CNN
 F 2 "" H 9200 3750 50  0001 C CNN
@@
 $EndComp
 $Comp
-L power:+3V3 #PWR043
+L power:+3V3 #PWR044
 U 1 1 5FAF359B
 P 9200 4450
-F 0 "#PWR043" H 9200 4300 50  0001 C CNN
+F 0 "#PWR044" H 9200 4300 50  0001 C CNN
 F 1 "+3V3" H 9200 4600 50  0000 C CNN
 F 2 "" H 9200 4450 50  0001 C CNN
@@
 Connection ~ 8500 4450
 $Comp
-L power:+3V3 #PWR041
+L power:+3V3 #PWR042
 U 1 1 5FAFFB75
 P 8550 5050
-F 0 "#PWR041" H 8550 4900 50  0001 C CNN
+F 0 "#PWR042" H 8550 4900 50  0001 C CNN
 F 1 "+3V3" H 8550 5200 50  0000 C CNN
 F 2 "" H 8550 5050 50  0001 C CNN
@@
 	1    0    0    -1
 $EndComp
+Text GLabel 7900 3650 0    50   Input ~ 0
+CAN-TX
 Text GLabel 7900 4350 0    50   Input ~ 0
-CAN-TX
-Text GLabel 7900 3650 0    50   Input ~ 0
 CAN-RX
 Text Notes 7950 3250 0    50   ~ 0
@@
 Wire Wire Line
 	6800 3600 6800 3700
+$Comp
+L Device:C_Small C13
+U 1 1 5FB35AC1
+P 8550 5150
+F 0 "C13" H 8450 5100 50  0000 R CNN
+F 1 "100nF" H 8450 5200 50  0000 R CNN
+F 2 "Capacitor_SMD:C_0603_1608Metric" H 8550 5150 50  0001 C CNN
+F 3 "~" H 8550 5150 50  0001 C CNN
+	1    8550 5150
+	-1   0    0    1
+$EndComp
+$Comp
+L power:GND #PWR040
+U 1 1 5FB364C5
+P 8550 5250
+F 0 "#PWR040" H 8550 5000 50  0001 C CNN
+F 1 "GND" H 8550 5100 50  0000 C CNN
+F 2 "" H 8550 5250 50  0001 C CNN
+F 3 "" H 8550 5250 50  0001 C CNN
+	1    8550 5250
+	1    0    0    -1
+$EndComp
+Connection ~ 8550 5050
+$Comp
+L Device:LED_Small D3
+U 1 1 5FAF24A0
+P 8900 3750
+F 0 "D3" H 8900 3985 50  0000 C CNN
+F 1 "CAN TX" H 8900 3894 50  0000 C CNN
+F 2 "LED_SMD:LED_0603_1608Metric" V 8900 3750 50  0001 C CNN
+F 3 "~" V 8900 3750 50  0001 C CNN
+	1    8900 3750
+	1    0    0    -1
+$EndComp
 $EndSCHEMATC

Commit message: :pencil: Add Mouser part numbers to BOM
Parts:
- C1, C5, C6: Mouser (none) -> 710-865230542002
- C10, C11, C12, C13, C7, C8, C9: Mouser (none) -> 710-885012206020
- C2, C3, C4: Mouser (none) -> 603-CC0603MRX6S5B226
- D1, D2, D4: Mouser (none) -> 710-150060RS75000
- D3: Mouser (none) -> 710-150060YS75000
- D5: Mouser (none) -> 863-SZNUP2105LT3G
- J1, J3: Mouser (none) -> 649-220327-C101B01LF
- J2, J4: Mouser (none) -> 571-6-534237-1
- J5: Mouser (none) -> 523-NY0210800000G
- J6, J7: Mouser (none) -> 571-5569284-1
- JP1: Mouser (none) -> 538-22-28-9034
- L1: Mouser (none) -> 81-B1047AS-4R7NP3
- R1, R2, R7, R8: Mouser (none) -> 603-AC0603JR-07160RL
- R3, R4, R5, R6: Mouser (none) -> 71-CRCW06030000Z0EAC
- SW1, SW2, SW3: Mouser (none) -> 667-EVQ-PE104K
- U2: Mouser (none) -> 621-AP63205WU-7
- U3: Mouser (none) -> 621-AP7365-33YG-13
- U4: Mouser (none) -> 595-LM358BIDR
- U5: Mouser (none) -> 726-IFX1050GVIOXUMA1
Other:
- note added: "5V 2A Buck Converter"
- note removed: "5V 2A LDO"
Changed lines of the file:
@@
 F 2 "Connector_RJ:RJ45_OST_PJ012-8P8CX_Vertical" V 10450 1475 50  0001 C CNN
 F 3 "~" V 10450 1475 50  0001 C CNN
+F 4 "571-5569284-1" H 10450 1450 50  0001 C CNN "Mouser"
 	1    10450 1450
 	-1   0    0    -1
@@
 F 2 "Connector_RJ:RJ45_OST_PJ012-8P8CX_Vertical" V 10450 2625 50  0001 C CNN
 F 3 "~" V 10450 2625 50  0001 C CNN
+F 4 "571-5569284-1" H 10450 2600 50  0001 C CNN "Mouser"
 	1    10450 2600
 	-1   0    0    -1
@@
 F 2 "Package_TO_SOT_SMD:TSOT-23-6" H 2000 5900 50  0001 C CNN
 F 3 "https://www.diodes.com/assets/Datasheets/AP63200-AP63201-AP63203-AP63205.pdf" H 2000 6800 50  0001 C CNN
+F 4 "621-AP63205WU-7" H 2000 6800 50  0001 C CNN "Mouser"
 	1    2000 6800
 	1    0    0    -1
@@
 F 2 "Inductor_SMD:L_7.3x7.3_H4.5" H 2650 6700 50  0001 C CNN
 F 3 "~" H 2650 6700 50  0001 C CNN
+F 4 "81-B1047AS-4R7NP3" V 2650 6700 50  0001 C CNN "Mouser"
 	1    2650 6700
 	0    -1   -1   0
@@
 F 2 "Capacitor_SMD:CP_Elec_5x5.3" H 1050 6850 50  0001 C CNN
 F 3 "~" H 1050 6850 50  0001 C CNN
+F 4 "710-865230542002" H 1050 6850 50  0001 C CNN "Mouser"
 	1    1050 6850
 	1    0    0    -1
@@
 F 2 "Capacitor_SMD:C_0603_1608Metric" H 2950 7000 50  0001 C CNN
 F 3 "~" H 2950 7000 50  0001 C CNN
+F 4 "603-CC0603MRX6S5B226" H 2950 7000 50  0001 C CNN "Mouser"
 	1    2950 7000
 	1    0    0    -1
@@
 F 2 "Capacitor_SMD:C_0603_1608Metric" H 2800 7000 50  0001 C CNN
 F 3 "~" H 2800 7000 50  0001 C CNN
+F 4 "603-CC0603MRX6S5B226" H 2800 7000 50  0001 C CNN "Mouser"
 	1    2800 7000
 	-1   0    0    1
@@
 F 2 "Capacitor_SMD:C_0603_1608Metric" H 2350 6350 50  0001 C CNN
 F 3 "~" H 2350 6350 50  0001 C CNN
+F 4 "603-CC0603MRX6S5B226" V 2350 6350 50  0001 C CNN "Mouser"
 	1    2350 6350
 	0    1    1    0
@@
 F 2 "Package_SO:SOIC-8_3.9x4.9mm_P1.27mm" H 8550 1600 50  0001 C CIN
 F 3 "http://www.nxp.com/documents/data_sheet/TJA1051.pdf" H 8550 2100 50  0001 C CNN
+F 4 "726-IFX1050GVIOXUMA1" H 8550 2100 50  0001 C CNN "Mouser"
 	1    8550 2100
 	1    0    0    -1
@@
 F 2 "Capacitor_SMD:C_0603_1608Metric" H 8350 1600 50  0001 C CNN
 F 3 "~" H 8350 1600 50  0001 C CNN
+F 4 "710-885012206020" V 8350 1600 50  0001 C CNN "Mouser"
 	1    8350 1600
 	0    1    1    0
@@
 F 2 "Capacitor_SMD:C_0603_1608Metric" H 7900 2300 50  0001 C CNN
 F 3 "~" H 7900 2300 50  0001 C CNN
+F 4 "710-885012206020" H 7900 2300 50  0001 C CNN "Mouser"
 	1    7900 2300
 	1    0    0    -1
@@
 F 2 "Connector_PinHeader_2.54mm:PinHeader_1x03_P2.54mm_Vertical" H 7450 5950 50  0001 C CNN
 F 3 "~" H 7450 5950 50  0001 C CNN
+F 4 "538-22-28-9034" H 7450 5950 50  0001 C CNN "Mouser"
 	1    7450 5950
 	1    0    0    -1
@@
 F 2 "TerminalBlock_Phoenix:TerminalBlock_Phoenix_PT-1,5-2-3.5-H_1x02_P3.50mm_Horizontal" H 8550 6250 50  0001 C CNN
 F 3 "~" H 8550 6250 50  0001 C CNN
+F 4 "523-NY0210800000G" H 8550 6250 50  0001 C CNN "Mouser"
 	1    8550 6250
 	1    0    0    1
@@
 F 2 "Package_TO_SOT_SMD:SOT-23" H 10425 3750 50  0001 L CNN
 F 3 "http://www.onsemi.com/pub_link/Collateral/NUP2105L-D.PDF" H 10325 3925 50  0001 C CNN
+F 4 "863-SZNUP2105LT3G" H 10200 3800 50  0001 C CNN "Mouser"
 	1    10200 3800
 	1    0    0    -1
@@
 F 2 "Package_SO:SOIC-8_3.9x4.9mm_P1.27mm" H 8200 3750 50  0001 C CNN
 F 3 "http://www.ti.com/lit/ds/symlink/lm2904-n.pdf" H 8200 3750 50  0001 C CNN
+F 4 "595-LM358BIDR" H 8200 3750 50  0001 C CNN "Mouser"
 	1    8200 3750
 	1    0    0    -1
@@
 F 2 "Package_SO:SOIC-8_3.9x4.9mm_P1.27mm" H 8200 4450 50  0001 C CNN
 F 3 "http://www.ti.com/lit/ds/symlink/lm2904-n.pdf" H 8200 4450 50  0001 C CNN
+F 4 "595-LM358BIDR" H 8200 4450 50  0001 C CNN "Mouser"
 	2    8200 4450
 	1    0    0    -1
@@
 F 2 "LED_SMD:LED_0603_1608Metric" V 8900 4450 50  0001 C CNN
 F 3 "~" V 8900 4450 50  0001 C CNN
+F 4 "710-150060RS75000" H 8900 4450 50  0001 C CNN "Mouser"
 	1    8900 4450
 	1    0    0    -1
@@
 F 2 "Resistor_SMD:R_0603_1608Metric" H 8650 3750 50  0001 C CNN
 F 3 "~" H 8650 3750 50  0001 C CNN
+F 4 "603-AC0603JR-07160RL" V 8650 3750 50  0001 C CNN "Mouser"
 	1    8650 3750
 	0    -1   -1   0
@@
 F 2 "Resistor_SMD:R_0603_1608Metric" H 8650 4450 50  0001 C CNN
 F 3 "~" H 8650 4450 50  0001 C CNN
+F 4 "603-AC0603JR-07160RL" V 8650 4450 50  0001 C CNN "Mouser"
 	1    8650 4450
 	0    -1   -1   0
@@
 CAN Activity LEDs
 Text Notes 1850 5900 0    50   ~ 0
-5V 2A LDO
+5V 2A Buck Converter
 $Comp
 L Components:ESP32-Module U1
@@
 F 2 "Button_Switch_SMD:SW_SPST_EVQPE1" H 4650 1550 50  0001 C CNN
 F 3 "~" H 4650 1550 50  0001 C CNN
+F 4 "667-EVQ-PE104K" H 4650 1350 50  0001 C CNN "Mouser"
 	1    4650 1350
 	1    0    0    -1
@@
 F 2 "Button_Switch_SMD:SW_SPST_EVQPE1" H 6350 1600 50  0001 C CNN
 F 3 "~" H 6350 1600 50  0001 C CNN
+F 4 "667-EVQ-PE104K" H 6350 1400 50  0001 C CNN "Mouser"
 	1    6350 1400
 	1    0    0    -1
@@
 F 2 "Resistor_SMD:R_0603_1608Metric" H 6050 1000 50  0001 C CNN
 F 3 "~" H 6050 1000 50  0001 C CNN
+F 4 "71-CRCW06030000Z0EAC" H 6050 1000 50  0001 C CNN "Mouser"
 	1    6050 1000
 	1    0    0    -1
@@
 F 2 "Button_Switch_SMD:SW_SPST_EVQPE1" H 6350 2650 50  0001 C CNN
 F 3 "~" H 6350 2650 50  0001 C CNN
+F 4 "667-EVQ-PE104K" H 6350 2450 50  0001 C CNN "Mouser"
 	1    6350 2450
 	1    0    0    -1
@@
 F 2 "Resistor_SMD:R_0603_1608Metric" H 6050 2250 50  0001 C CNN
 F 3 "~" H 6050 2250 50  0001 C CNN
+F 4 "71-CRCW06030000Z0EAC" H 6050 2250 50  0001 C CNN "Mouser"
 	1    6050 2250
 	1    0    0    -1
@@
 F 2 "Capacitor_SMD:C_0603_1608Metric" H 6050 2650 50  0001 C CNN
 F 3 "~" H 6050 2650 50  0001 C CNN
+F 4 "710-885012206020" H 6050 2650 50  0001 C CNN "Mouser"
 	1    6050 2650
 	-1   0    0    1
@@
 F 2 "Capacitor_SMD:C_0603_1608Metric" H 6050 1600 50  0001 C CNN
 F 3 "~" H 6050 1600 50  0001 C CNN
+F 4 "710-885012206020" H 6050 1600 50  0001 C CNN "Mouser"
 	1    6050 1600
 	-1   0    0    1
@@
 F 2 "TerminalBlock_Phoenix:TerminalBlock_Phoenix_PT-1,5-10-3.5-H_1x10_P3.50mm_Horizontal" H 3900 4150 50  0001 C CNN
 F 3 "~" H 3900 4150 50  0001 C CNN
+F 4 "649-220327-C101B01LF" H 3900 4150 50  0001 C CNN "Mouser"
 	1    3900 4150
 	1    0    0    1
@@
 F 2 "TerminalBlock_Phoenix:TerminalBlock_Phoenix_PT-1,5-10-3.5-H_1x10_P3.50mm_Horizontal" H 1250 4000 50  0001 C CNN
 F 3 "~" H 1250 4000 50  0001 C CNN
+F 4 "649-220327-C101B01LF" H 1250 4000 50  0001 C CNN "Mouser"
 	1    1250 4000
 	1    0    0    -1
@@
 F 2 "LED_SMD:LED_0603_1608Metric" V 4600 1950 50  0001 C CNN
 F 3 "~" V 4600 1950 50  0001 C CNN
+F 4 "710-150060RS75000" H 4600 1950 50  0001 C CNN "Mouser"
 	1    4600 1950
 	1    0    0    -1
@@
 F 2 "Resistor_SMD:R_0603_1608Metric" H 4350 1950 50  0001 C CNN
 F 3 "~" H 4350 1950 50  0001 C CNN
+F 4 "603-AC0603JR-07160RL" V 4350 1950 50  0001 C CNN "Mouser"
 	1    4350 1950
 	0    -1   -1   0
@@
 F 2 "LED_SMD:LED_0603_1608Metric" V 4600 2300 50  0001 C CNN
 F 3 "~" V 4600 2300 50  0001 C CNN
+F 4 "710-150060RS75000" H 4600 2300 50  0001 C CNN "Mouser"
 	1    4600 2300
 	1    0    0    -1
@@
 F 2 "Resistor_SMD:R_0603_1608Metric" H 4350 2300 50  0001 C CNN
 F 3 "~" H 4350 2300 50  0001 C CNN
+F 4 "603-AC0603JR-07160RL" V 4350 2300 50  0001 C CNN "Mouser"
 	1    4350 2300
 	0    -1   -1   0
@@
 F 2 "Package_TO_SOT_SMD:SOT-223-3_TabPin2" H 4850 6800 50  0001 C CNN
 F 3 "http://www.onsemi.com/pub_link/Collateral/NCP1117-D.PDF" H 4950 6350 50  0001 C CNN
+F 4 "621-AP7365-33YG-13" H 4850 6600 50  0001 C CNN "Mouser"
 	1    4850 6600
 	1    0    0    -1
@@
 F 2 "Capacitor_SMD:CP_Elec_5x5.3" H 4450 6800 50  0001 C CNN
 F 3 "~" H 4450 6800 50  0001 C CNN
+F 4 "710-865230542002" H 4450 6800 50  0001 C CNN "Mouser"
 	1    4450 6800
 	1    0    0    -1
@@
 F 2 "Capacitor_SMD:CP_Elec_5x5.3" H 5250 6800 50  0001 C CNN
 F 3 "~" H 5250 6800 50  0001 C CNN
+F 4 "710-865230542002" H 5250 6800 50  0001 C CNN "Mouser"
 	1    5250 6800
 	1    0    0    -1
@@
 F 2 "Connector_PinSocket_2.54mm:PinSocket_1x13_P2.54mm_Vertical" H 4950 4050 50  0001 C CNN
 F 3 "~" H 4950 4050 50  0001 C CNN
+F 4 "571-6-534237-1" H 4950 4050 50  0001 C CNN "Mouser"
 	1    4950 4050
 	1    0    0    -1
@@
 F 2 "Connector_PinSocket_2.54mm:PinSocket_1x13_P2.54mm_Vertical" H 2450 4050 50  0001 C CNN
 F 3 "~" H 2450 4050 50  0001 C CNN
+F 4 "571-6-534237-1" H 2450 4050 50  0001 C CNN "Mouser"
 	1    2450 4050
 	1    0    0    -1
@@
 F 2 "Resistor_SMD:R_0603_1608Metric" H 6100 3400 50  0001 C CNN
 F 3 "~" H 6100 3400 50  0001 C CNN
+F 4 "71-CRCW06030000Z0EAC" H 6100 3400 50  0001 C CNN "Mouser"
 	1    6100 3400
 	1    0    0    -1
@@
 F 2 "Capacitor_SMD:C_0603_1608Metric" H 6100 3800 50  0001 C CNN
 F 3 "~" H 6100 3800 50  0001 C CNN
+F 4 "710-885012206020" H 6100 3800 50  0001 C CNN "Mouser"
 	1    6100 3800
 	-1   0    0    1
@@
 F 2 "Resistor_SMD:R_0603_1608Metric" H 6800 3400 50  0001 C CNN
 F 3 "~" H 6800 3400 50  0001 C CNN
+F 4 "71-CRCW06030000Z0EAC" H 6800 3400 50  0001 C CNN "Mouser"
 	1    6800 3400
 	1    0    0    -1
@@
 F 2 "Capacitor_SMD:C_0603_1608Metric" H 6800 3800 50  0001 C CNN
 F 3 "~" H 6800 3800 50  0001 C CNN
+F 4 "710-885012206020" H 6800 3800 50  0001 C CNN "Mouser"
 	1    6800 3800
 	-1   0    0    1
@@
 F 2 "Capacitor_SMD:C_0603_1608Metric" H 8550 5150 50  0001 C CNN
 F 3 "~" H 8550 5150 50  0001 C CNN
+F 4 "710-885012206020" H 8550 5150 50  0001 C CNN "Mouser"
 	1    8550 5150
 	-1   0    0    1
@@
 F 2 "LED_SMD:LED_0603_1608Metric" V 8900 3750 50  0001 C CNN
 F 3 "~" V 8900 3750 50  0001 C CNN
+F 4 "710-150060YS75000" H 8900 3750 50  0001 C CNN "Mouser"
 	1    8900 3750
 	1    0    0    -1

Commit message: :pencil: Corrections to part numbers
* C2 should have been 100nF and not 22uF
* U3 needs to be able to provide 1A and not 600mA.
Parts:
- C2: value 22uF -> 100nF; Mouser 603-CC0603MRX6S5B226 -> 710-885012206020
- U3: value NCP1117 -> AP2114-3.3; Mouser 621-AP7365-33YG-13 -> AP2114HA-3.3TRG1
Changed lines of the file:
@@
 Sheet 1 1
 Title "ESP32 IO Board"
-Date "2020-11-16"
+Date "2020-11-18"
 Rev "1.0"
 Comp ""
@@
 P 2350 6350
 F 0 "C2" V 2121 6350 50  0000 C CNN
-F 1 "22uF" V 2212 6350 50  0000 C CNN
+F 1 "100nF" V 2212 6350 50  0000 C CNN
 F 2 "Capacitor_SMD:C_0603_1608Metric" H 2350 6350 50  0001 C CNN
 F 3 "~" H 2350 6350 50  0001 C CNN
-F 4 "603-CC0603MRX6S5B226" V 2350 6350 50  0001 C CNN "Mouser"
+F 4 "710-885012206020" V 2350 6350 50  0001 C CNN "Mouser"
 	1    2350 6350
 	0    1    1    0
@@
 P 4850 6600
 F 0 "U3" H 4850 6842 50  0000 C CNN
-F 1 "NCP1117" H 4850 6751 50  0000 C CNN
+F 1 "AP2114-3.3" H 4850 6751 50  0000 C CNN
 F 2 "Package_TO_SOT_SMD:SOT-223-3_TabPin2" H 4850 6800 50  0001 C CNN
 F 3 "http://www.onsemi.com/pub_link/Collateral/NCP1117-D.PDF" H 4950 6350 50  0001 C CNN
-F 4 "621-AP7365-33YG-13" H 4850 6600 50  0001 C CNN "Mouser"
+F 4 "AP2114HA-3.3TRG1" H 4850 6600 50  0001 C CNN "Mouser"
 	1    4850 6600
 	1    0    0    -1

Commit message: :pencil: Update schematic with a few part alternatives
Parts:
- J2, J4: Mouser 571-6-534237-1 -> 571-6-534237-1 or 992-13FX1-254MM
- J6, J7: Mouser 571-5569284-1 -> 571-5569284-1 or 534-949 or 493-HCJV1-812UK
Changed lines of the file:
@@
 F 2 "Connector_RJ:RJ45_OST_PJ012-8P8CX_Vertical" V 10450 1475 50  0001 C CNN
 F 3 "~" V 10450 1475 50  0001 C CNN
-F 4 "571-5569284-1" H 10450 1450 50  0001 C CNN "Mouser"
+F 4 "571-5569284-1 or 534-949 or 493-HCJV1-812UK" H 10450 1450 50  0001 C CNN "Mouser"
 	1    10450 1450
 	-1   0    0    -1
@@
 F 2 "Connector_RJ:RJ45_OST_PJ012-8P8CX_Vertical" V 10450 2625 50  0001 C CNN
 F 3 "~" V 10450 2625 50  0001 C CNN
-F 4 "571-5569284-1" H 10450 2600 50  0001 C CNN "Mouser"
+F 4 "571-5569284-1 or 534-949 or 493-HCJV1-812UK" H 10450 2600 50  0001 C CNN "Mouser"
 	1    10450 2600
 	-1   0    0    -1
@@
 F 2 "Connector_PinSocket_2.54mm:PinSocket_1x13_P2.54mm_Vertical" H 4950 4050 50  0001 C CNN
 F 3 "~" H 4950 4050 50  0001 C CNN
-F 4 "571-6-534237-1" H 4950 4050 50  0001 C CNN "Mouser"
+F 4 "571-6-534237-1 or 992-13FX1-254MM" H 4950 4050 50  0001 C CNN "Mouser"
 	1    4950 4050
 	1    0    0    -1
@@
 F 2 "Connector_PinSocket_2.54mm:PinSocket_1x13_P2.54mm_Vertical" H 2450 4050 50  0001 C CNN
 F 3 "~" H 2450 4050 50  0001 C CNN
-F 4 "571-6-534237-1" H 2450 4050 50  0001 C CNN "Mouser"
+F 4 "571-6-534237-1 or 992-13FX1-254MM" H 2450 4050 50  0001 C CNN "Mouser"
 	1    2450 4050
 	1    0    0    -1

Commit message: :pencil: Add Fiducials to PCB :pencil: Adjust LED colors so they are not all red
Parts:
- added FID1, FID2, FID3: Fiducial, Fiducial:Fiducial_0.5mm_Mask1mm, symbol Mechanical:Fiducial
- D1: Mouser 710-150060RS75000 -> 710-150060VS55040
- D2, D4: Mouser 710-150060RS75000 -> 710-150060AS75000
Changed lines of the file:
@@
 Sheet 1 1
 Title "ESP32 IO Board"
-Date "2020-11-18"
+Date "2020-11-19"
 Rev "1.0"
 Comp ""
@@
 F 2 "LED_SMD:LED_0603_1608Metric" V 8900 4450 50  0001 C CNN
 F 3 "~" V 8900 4450 50  0001 C CNN
-F 4 "710-150060RS75000" H 8900 4450 50  0001 C CNN "Mouser"
+F 4 "710-150060AS75000" H 8900 4450 50  0001 C CNN "Mouser"
 	1    8900 4450
 	1    0    0    -1
@@
 F 2 "LED_SMD:LED_0603_1608Metric" V 4600 1950 50  0001 C CNN
 F 3 "~" V 4600 1950 50  0001 C CNN
-F 4 "710-150060RS75000" H 4600 1950 50  0001 C CNN "Mouser"
+F 4 "710-150060VS55040" H 4600 1950 50  0001 C CNN "Mouser"
 	1    4600 1950
 	1    0    0    -1
@@
 F 2 "LED_SMD:LED_0603_1608Metric" V 4600 2300 50  0001 C CNN
 F 3 "~" V 4600 2300 50  0001 C CNN
-F 4 "710-150060RS75000" H 4600 2300 50  0001 C CNN "Mouser"
+F 4 "710-150060AS75000" H 4600 2300 50  0001 C CNN "Mouser"
 	1    4600 2300
 	1    0    0    -1
@@
 	1    0    0    -1
 $EndComp
+$Comp
+L Mechanical:Fiducial FID3
+U 1 1 5FB6ED3B
+P 5750 7650
+F 0 "FID3" H 5835 7696 50  0000 L CNN
+F 1 "Fiducial" H 5835 7605 50  0000 L CNN
+F 2 "Fiducial:Fiducial_0.5mm_Mask1mm" H 5750 7650 50  0001 C CNN
+F 3 "~" H 5750 7650 50  0001 C CNN
+	1    5750 7650
+	1    0    0    -1
+$EndComp
+$Comp
+L Mechanical:Fiducial FID2
+U 1 1 5FB6F6CE
+P 5750 7450
+F 0 "FID2" H 5835 7496 50  0000 L CNN
+F 1 "Fiducial" H 5835 7405 50  0000 L CNN
+F 2 "Fiducial:Fiducial_0.5mm_Mask1mm" H 5750 7450 50  0001 C CNN
+F 3 "~" H 5750 7450 50  0001 C CNN
+	1    5750 7450
+	1    0    0    -1
+$EndComp
+$Comp
+L Mechanical:Fiducial FID1
+U 1 1 5FB70D5E
+P 5750 7250
+F 0 "FID1" H 5835 7296 50  0000 L CNN
+F 1 "Fiducial" H 5835 7205 50  0000 L CNN
+F 2 "Fiducial:Fiducial_0.5mm_Mask1mm" H 5750 7250 50  0001 C CNN
+F 3 "~" H 5750 7250 50  0001 C CNN
+	1    5750 7250
+	1    0    0    -1
+$EndComp

Commit message: :pencil: Correct BOM reference for 3v3 LDO
Parts:
- U3: Mouser AP2114HA-3.3TRG1 -> 621-AP2114H-3.3TRG1
Changed lines of the file:
@@
 F 2 "Package_TO_SOT_SMD:SOT-223-3_TabPin2" H 4850 6800 50  0001 C CNN
 F 3 "http://www.onsemi.com/pub_link/Collateral/NCP1117-D.PDF" H 4950 6350 50  0001 C CNN
-F 4 "AP2114HA-3.3TRG1" H 4850 6600 50  0001 C CNN "Mouser"
+F 4 "621-AP2114H-3.3TRG1" H 4850 6600 50  0001 C CNN "Mouser"
 	1    4850 6600
 	1    0    0    -1

Commit message: :pencil: PCB BOM update
Parts:
- J5: Mouser 523-NY0210800000G -> 651-1984617
Changed lines of the file:
@@
 Sheet 1 1
 Title "ESP32 IO Board"
-Date "2020-11-19"
+Date "2020-12-04"
 Rev "1.0"
 Comp ""
@@
 F 2 "TerminalBlock_Phoenix:TerminalBlock_Phoenix_PT-1,5-2-3.5-H_1x02_P3.50mm_Horizontal" H 8550 6250 50  0001 C CNN
 F 3 "~" H 8550 6250 50  0001 C CNN
-F 4 "523-NY0210800000G" H 8550 6250 50  0001 C CNN "Mouser"
+F 4 "651-1984617" H 8550 6250 50  0001 C CNN "Mouser"
 	1    8550 6250
 	1    0    0    1
