File: pcb/pcb.kicad_pcb (KiCad board)
At the start: 4 copper layers, 61 x 81 mm, 52 parts, among them J1 LEFT, J2 LEFT-EXT, J3 RIGHT, J4 RIGHT-EXT, J5 EXT POWER, J6 RJ45, J7 RJ45, SW1 Reset, SW2 Factory Reset, SW3 User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

Commit message: Adding one additional GND via to v1.1 PCB, add position file.
Routing:
- net GND: track 27.5 -> 28.4 mm, vias 18 -> 19
Other:
- board text added: "Activity"
- board text added: "WiFi"
- board text removed: "Node Activity"
- board text removed: "WiFi on"
Changed lines of the file:
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@@
   (title_block
     (title "ESP32 OpenLCB IO Board")
-    (date "2022-09-17")
+    (date "2022-09-29")
     (rev "1.1")
   )
@@
     (effects (font (size 1.5 1.5) (thickness 0.3)) (justify left))
   )
-  (gr_text "WiFi on" (at 160.16 57.19) (layer "F.SilkS")
+  (gr_text "WiFi" (at 160.16 57.19) (layer "F.SilkS")
     (effects (font (size 1 1) (thickness 0.15)) (justify left))
   )
@@
     (effects (font (size 1.5 1.5) (thickness 0.2)))
   )
-  (gr_text "Node\nActivity" (at 160.16 59.55) (layer "F.SilkS")
+  (gr_text "Activity" (at 160.16 58.99) (layer "F.SilkS")
     (effects (font (size 1 1) (thickness 0.15)) (justify left))
   )
@@
   (segment (start 145.63 98.934142) (end 145.63 100.85) (width 0.5) (layer "F.Cu") (net 1))
   (segment (start 134.845 120.695) (end 134.85 120.7) (width 0.5) (layer "F.Cu") (net 1))
+  (segment (start 127.68 61.32) (end 127.68 62.22) (width 0.5) (layer "F.Cu") (net 1))
   (segment (start 145.64 98.91) (end 145.65 98.9) (width 0.5) (layer "F.Cu") (net 1))
   (segment (start 132.715 107.135) (end 132.73 107.12) (width 0.5) (layer "F.Cu") (net 1))
@@
   (segment (start 109.684142 114.12) (end 110.57 114.12) (width 0.5) (layer "F.Cu") (net 1))
   (segment (start 122.417071 103.56) (end 123.85 103.56) (width 0.5) (layer "F.Cu") (net 1))
+  (segment (start 127.68 62.22) (end 127.65 62.25) (width 0.5) (layer "F.Cu") (net 1))
   (segment (start 133.581 111.610468) (end 133.581 113.568) (width 0.5) (layer "F.Cu") (net 1))
   (segment (start 109.95 100.2) (end 109.95 101.69) (width 0.5) (layer "F.Cu") (net 1))
@@
   (via (at 129.6 99.25) (size 0.6) (drill 0.4) (layers "F.Cu" "B.Cu") (net 1))
   (via (at 111.45 57.4) (size 0.6) (drill 0.4) (layers "F.Cu" "B.Cu") (net 1))
+  (via (at 127.65 62.25) (size 0.6) (drill 0.4) (layers "F.Cu" "B.Cu") (net 1))
   (via (at 109.65 114.1) (size 0.6) (drill 0.4) (layers "F.Cu" "B.Cu") (net 1))
   (arc (start 134.845 120.695) (mid 134.839461 120.691299) (end 134.832928 120.69) (width 0.5) (layer "F.Cu") (net 1))
