File: pcb-servo/pcb-servo.sch (KiCad schematic (older format))
At the start: 25 parts, among them J1 PWM, J10 PWM, J11 PWM, J12 PWM, J13 PWM, J14 PWM, J15 PWM, J16 PWM, J17 LEFT-EXT, J18 RIGHT-EXT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

Commit message: :pencil: Corrections to part numbers
Parts:
- C1: LCSC (none) -> C85713; Mouser 81-GRM033R60J105ME2D -> 187-CL10A106MQ8NNNC
- R1: LCSC (none) -> C98220
- R2: LCSC (none) -> C95331
- RN1, RN2: LCSC (none) -> C422184
- U2: LCSC (none) -> C128835
Changed lines of the file:
@@
 F 3 "~" H 1450 1700 50  0001 C CNN
 F 4 "71-CRCW06030000Z0EAC" V 1450 1700 50  0001 C CNN "Mouser"
+F 5 "C98220" V 1450 1700 50  0001 C CNN "LCSC"
 	1    1450 1700
 	0    1    1    0
@@
 F 2 "Capacitor_SMD:C_0603_1608Metric" H 1500 3800 50  0001 C CNN
 F 3 "https://www.mouser.com/datasheet/2/281/1/GRM033R60J105MEA2_61A-1981777.pdf" H 1500 3800 50  0001 C CNN
-F 4 "81-GRM033R60J105ME2D" H 1500 3800 50  0001 C CNN "Mouser"
+F 4 "187-CL10A106MQ8NNNC" H 1500 3800 50  0001 C CNN "Mouser"
+F 5 "C85713" H 1500 3800 50  0001 C CNN "LCSC"
 	1    1500 3800
 	1    0    0    -1
@@
 F 3 "https://www.mouser.com/datasheet/2/54/CATCAY-777361.pdf" H 3150 1800 50  0001 C CNN
 F 4 "652-CAY16-221J8LF" V 3150 1800 50  0001 C CNN "Mouser"
+F 5 "C422184" V 3150 1800 50  0001 C CNN "LCSC"
 	1    3150 1800
 	0    -1   1    0
@@
 F 3 "https://www.mouser.com/datasheet/2/54/CATCAY-777361.pdf" H 3150 2500 50  0001 C CNN
 F 4 "652-CAY16-221J8LF" V 3150 2500 50  0001 C CNN "Mouser"
+F 5 "C422184" V 3150 2500 50  0001 C CNN "LCSC"
 	1    3150 2500
 	0    1    -1   0
@@
 F 3 "https://www.mouser.com/datasheet/2/302/PCA9306-1127635.pdf" H 4750 2600 50  0001 C CNN
 F 4 "771-PCA9306DP1-G" H 5050 2150 50  0001 C CNN "Mouser"
+F 5 "C128835" H 5050 2150 50  0001 C CNN "LCSC"
 	1    5050 2150
 	1    0    0    -1
@@
 F 3 "https://www.mouser.com/datasheet/2/427/crcwce3-1762584.pdf" H 5500 1800 50  0001 C CNN
 F 4 "71-CRCW0603200KFKEAC" H 5500 1800 50  0001 C CNN "Mouser"
+F 5 "C95331" H 5500 1800 50  0001 C CNN "LCSC"
 	1    5500 1800
 	1    0    0    -1

Commit message: :pencil: adjust PCB to use a cut out instead of solid panel
Parts:
- RN1, RN2: footprint Resistor_SMD:R_Cat16-8 -> Resistor_SMD:R_Array_Convex_8x0602
Changed lines of the file:
@@
 F 0 "RN1" V 2533 1800 50  0000 C CNN
 F 1 "220R" V 2624 1800 50  0000 C CNN
-F 2 "Resistor_SMD:R_Cat16-8" V 3625 1800 50  0001 C CNN
+F 2 "Resistor_SMD:R_Array_Convex_8x0602" V 3625 1800 50  0001 C CNN
 F 3 "https://www.mouser.com/datasheet/2/54/CATCAY-777361.pdf" H 3150 1800 50  0001 C CNN
 F 4 "652-CAY16-221J8LF" V 3150 1800 50  0001 C CNN "Mouser"
@@
 F 0 "RN2" V 2550 2500 50  0000 C CNN
 F 1 "220R" V 2650 2500 50  0000 C CNN
-F 2 "Resistor_SMD:R_Cat16-8" V 3625 2500 50  0001 C CNN
+F 2 "Resistor_SMD:R_Array_Convex_8x0602" V 3625 2500 50  0001 C CNN
 F 3 "https://www.mouser.com/datasheet/2/54/CATCAY-777361.pdf" H 3150 2500 50  0001 C CNN
 F 4 "652-CAY16-221J8LF" V 3150 2500 50  0001 C CNN "Mouser"

Commit message: :tractor: Update with current PCB in testing.
Parts:
- added C2, C3, C4, C5: DNP, Capacitor_THT:CP_Radial_D8.0mm_P3.50mm, symbol Device:CP1_Small
Connections:
- net +5V: now also C2.1, C3.1, C4.1, C5.1
- net GND: now also C2.2, C3.2, C4.2, C5.2
Changed lines of the file:
@@
 IO8
 $Comp
-L power:GND #PWR043
+L power:GND #PWR051
 U 1 1 5FBB3A82
 P 10400 1100
-F 0 "#PWR043" H 10400 850 50  0001 C CNN
+F 0 "#PWR051" H 10400 850 50  0001 C CNN
 F 1 "GND" V 10405 972 50  0000 R CNN
 F 2 "" H 10400 1100 50  0001 C CNN
@@
 $EndComp
 $Comp
-L power:+3V3 #PWR044
+L power:+3V3 #PWR052
 U 1 1 5FBB3A8C
 P 10400 1200
-F 0 "#PWR044" H 10400 1050 50  0001 C CNN
+F 0 "#PWR052" H 10400 1050 50  0001 C CNN
 F 1 "+3V3" V 10400 1450 50  0000 C CNN
 F 2 "" H 10400 1200 50  0001 C CNN
@@
 IO14
 $Comp
-L power:GND #PWR041
+L power:GND #PWR049
 U 1 1 5FBB7FC6
 P 9400 2200
-F 0 "#PWR041" H 9400 1950 50  0001 C CNN
+F 0 "#PWR049" H 9400 1950 50  0001 C CNN
 F 1 "GND" V 9405 2072 50  0000 R CNN
 F 2 "" H 9400 2200 50  0001 C CNN
@@
 IO15
 $Comp
-L power:VCC #PWR042
+L power:VCC #PWR050
 U 1 1 5FBD40F3
 P 10400 1000
-F 0 "#PWR042" H 10400 850 50  0001 C CNN
+F 0 "#PWR050" H 10400 850 50  0001 C CNN
 F 1 "VCC" V 10400 1200 50  0000 C CNN
 F 2 "" H 10400 1000 50  0001 C CNN
@@
 I2C_SDA
 $Comp
-L power:+5V #PWR040
+L power:+5V #PWR048
 U 1 1 5FBE081B
 P 9400 2100
-F 0 "#PWR040" H 9400 1950 50  0001 C CNN
+F 0 "#PWR048" H 9400 1950 50  0001 C CNN
 F 1 "+5V" V 9400 2300 50  0000 C CNN
 F 2 "" H 9400 2100 50  0001 C CNN
@@
 $EndComp
 $Comp
-L power:GND #PWR038
+L power:GND #PWR044
 U 1 1 601DEBDB
 P 5050 2650
-F 0 "#PWR038" H 5050 2400 50  0001 C CNN
+F 0 "#PWR044" H 5050 2400 50  0001 C CNN
 F 1 "GND" H 5100 2500 50  0000 R CNN
 F 2 "" H 5050 2650 50  0001 C CNN
@@
 $EndComp
 $Comp
-L power:+5V #PWR039
+L power:+5V #PWR047
 U 1 1 601DF46E
 P 5500 1550
-F 0 "#PWR039" H 5500 1400 50  0001 C CNN
+F 0 "#PWR047" H 5500 1400 50  0001 C CNN
 F 1 "+5V" H 5500 1700 50  0000 C CNN
 F 2 "" H 5500 1550 50  0001 C CNN
@@
 $EndComp
 $Comp
-L power:+3V3 #PWR037
+L power:+3V3 #PWR043
 U 1 1 601E049E
 P 4950 1650
-F 0 "#PWR037" H 4950 1500 50  0001 C CNN
+F 0 "#PWR043" H 4950 1500 50  0001 C CNN
 F 1 "+3V3" H 4950 1800 50  0000 C CNN
 F 2 "" H 4950 1650 50  0001 C CNN
@@
 Text GLabel 1550 1500 0    50   BiDi ~ 0
 5V_I2C_SDA
+$Comp
+L Device:CP1_Small C3
+U 1 1 60FB1D5E
+P 1900 5050
+F 0 "C3" H 1991 5096 50  0000 L CNN
+F 1 "DNP" H 1991 5005 50  0000 L CNN
+F 2 "Capacitor_THT:CP_Radial_D8.0mm_P3.50mm" H 1900 5050 50  0001 C CNN
+F 3 "~" H 1900 5050 50  0001 C CNN
+	1    1900 5050
+	1    0    0    -1
+$EndComp
+$Comp
+L power:+5V #PWR039
+U 1 1 60FB2133
+P 1900 4950
+F 0 "#PWR039" H 1900 4800 50  0001 C CNN
+F 1 "+5V" H 1900 5100 50  0000 C CNN
+F 2 "" H 1900 4950 50  0001 C CNN
+F 3 "" H 1900 4950 50  0001 C CNN
+	1    1900 4950
+	1    0    0    -1
+$EndComp
+$Comp
+L power:GND #PWR040
+U 1 1 60FB2DE9
+P 1900 5150
+F 0 "#PWR040" H 1900 4900 50  0001 C CNN
+F 1 "GND" H 2000 5000 50  0000 R CNN
+F 2 "" H 1900 5150 50  0001 C CNN
+F 3 "" H 1900 5150 50  0001 C CNN
+	1    1900 5150
+	1    0    0    -1
+$EndComp
+$Comp
+L Device:CP1_Small C2
+U 1 1 60FB3922
+P 1550 5050
+F 0 "C2" H 1641 5096 50  0000 L CNN
+F 1 "DNP" H 1641 5005 50  0000 L CNN
+F 2 "Capacitor_THT:CP_Radial_D8.0mm_P3.50mm" H 1550 5050 50  0001 C CNN
+F 3 "~" H 1550 5050 50  0001 C CNN
+	1    1550 5050
+	1    0    0    -1
+$EndComp
+$Comp
+L power:+5V #PWR037
+U 1 1 60FB3F72
+P 1550 4950
+F 0 "#PWR037" H 1550 4800 50  0001 C CNN
+F 1 "+5V" H 1550 5100 50  0000 C CNN
+F 2 "" H 1550 4950 50  0001 C CNN
+F 3 "" H 1550 4950 50  0001 C CNN
+	1    1550 4950
+	1    0    0    -1
+$EndComp
+$Comp
+L power:GND #PWR038
+U 1 1 60FB3F7C
+P 1550 5150
+F 0 "#PWR038" H 1550 4900 50  0001 C CNN
+F 1 "GND" H 1650 5000 50  0000 R CNN
+F 2 "" H 1550 5150 50  0001 C CNN
+F 3 "" H 1550 5150 50  0001 C CNN
+	1    1550 5150
+	1    0    0    -1
+$EndComp
+$Comp
+L Device:CP1_Small C5
+U 1 1 60FBE754
+P 2600 5050
+F 0 "C5" H 2691 5096 50  0000 L CNN
+F 1 "DNP" H 2691 5005 50  0000 L CNN
+F 2 "Capacitor_THT:CP_Radial_D8.0mm_P3.50mm" H 2600 5050 50  0001 C CNN
+F 3 "~" H 2600 5050 50  0001 C CNN
+	1    2600 5050
+	1    0    0    -1
+$EndComp
+$Comp
+L power:+5V #PWR045
+U 1 1 60FBEDD8
+P 2600 4950
+F 0 "#PWR045" H 2600 4800 50  0001 C CNN
+F 1 "+5V" H 2600 5100 50  0000 C CNN
+F 2 "" H 2600 4950 50  0001 C CNN
+F 3 "" H 2600 4950 50  0001 C CNN
+	1    2600 4950
+	1    0    0    -1
+$EndComp
+$Comp
+L power:GND #PWR046
+U 1 1 60FBEDE2
+P 2600 5150
+F 0 "#PWR046" H 2600 4900 50  0001 C CNN
+F 1 "GND" H 2700 5000 50  0000 R CNN
+F 2 "" H 2600 5150 50  0001 C CNN
+F 3 "" H 2600 5150 50  0001 C CNN
+	1    2600 5150
+	1    0    0    -1
+$EndComp
+$Comp
+L Device:CP1_Small C4
+U 1 1 60FBEDEC
+P 2250 5050
+F 0 "C4" H 2341 5096 50  0000 L CNN
+F 1 "DNP" H 2341 5005 50  0000 L CNN
+F 2 "Capacitor_THT:CP_Radial_D8.0mm_P3.50mm" H 2250 5050 50  0001 C CNN
+F 3 "~" H 2250 5050 50  0001 C CNN
+	1    2250 5050
+	1    0    0    -1
+$EndComp
+$Comp
+L power:+5V #PWR041
+U 1 1 60FBEDF6
+P 2250 4950
+F 0 "#PWR041" H 2250 4800 50  0001 C CNN
+F 1 "+5V" H 2250 5100 50  0000 C CNN
+F 2 "" H 2250 4950 50  0001 C CNN
+F 3 "" H 2250 4950 50  0001 C CNN
+	1    2250 4950
+	1    0    0    -1
+$EndComp
+$Comp
+L power:GND #PWR042
+U 1 1 60FBEE00
+P 2250 5150
+F 0 "#PWR042" H 2250 4900 50  0001 C CNN
+F 1 "GND" H 2350 5000 50  0000 R CNN
+F 2 "" H 2250 5150 50  0001 C CNN
+F 3 "" H 2250 5150 50  0001 C CNN
+	1    2250 5150
+	1    0    0    -1
+$EndComp
 $EndSCHEMATC
